Commit message: Updated robot xacro

File: encRobo/src/enc/description/robot_core.xacro (robot description, xacro)
@@ -10,5 +10,5 @@
     <xacro:property name="wheel_mass" value="0.335"/>
     <xacro:property name="wheel_offset_x" value="0.03"/>
-    <xacro:property name="wheel_offset_y" value="0.091"/>
+    <xacro:property name="wheel_offset_y" value="0.182"/>
     <xacro:property name="wheel_offset_z" value="0.01"/>
     <xacro:property name="caster_wheel_radius" value="0.045"/>
@@ -100,5 +100,5 @@
         <child link="right_wheel"/>
         <origin xyz="0 ${-wheel_offset_y} 0" rpy="${pi/2} 0 0" />
-        <axis xyz="0 0 -1"/>
+        <axis xyz="0 0 1"/>
     </joint>
     <link name="right_wheel">
